File: Digitaler_Wuerfel.kicad_pcb (KiCad board)
At the start: 2 copper layers, 32 parts, among them J1 Conn_01x03_Pin, J2 Conn_02x03_Odd_Even, U1 74HC595, U2 74HC595, U3 ATmega328PB-A, U4 LM7805_TO220

Commit message: Started tracing
Parts:
- removed the U4 at (40.5, 58.7)
- added C1: 470pF, Capacitor_SMD:C_0805_2012Metric_Pad1.18x1.45mm_HandSolder, F.Cu at (114.5, 73.5)
- added C2: 0.1uF, Capacitor_SMD:C_0805_2012Metric_Pad1.18x1.45mm_HandSolder, F.Cu at (112.0, 65.0)
- added C7: 470pF, Capacitor_SMD:C_0805_2012Metric_Pad1.18x1.45mm_HandSolder, F.Cu at (100.5, 99.0)
- added C8: 2.2uF, Capacitor_Tantalum_SMD:CP_EIA-3528-21_Kemet-B_Pad1.50x2.35mm_HandSolder, F.Cu at (95.4, 99.0)
- added D1: D_Schottky, Diode_SMD:D_SOD-323_HandSoldering, F.Cu at (100.5, 104.5)
- added GND: TestPoint_Probe, TestPoint:TestPoint_Pad_D2.0mm, F.Cu at (89.0, 105.5)
- added Q1: 2N3904, Package_TO_SOT_THT:TO-92_Inline, F.Cu at (114.5, 78.5)
- added R1: 200k, Resistor_SMD:R_0805_2012Metric_Pad1.20x1.40mm_HandSolder, F.Cu at (113.5, 82.0)
- added R11: 1k, Resistor_SMD:R_0805_2012Metric_Pad1.20x1.40mm_HandSolder, F.Cu at (108.0, 78.5)
- added R12: 1k, Resistor_SMD:R_0805_2012Metric_Pad1.20x1.40mm_HandSolder, F.Cu at (111.5, 78.5)
- added SW1: SW_Push, Button_Switch_THT:SW_PUSH-12mm_Wuerth-430476085716, F.Cu at (139.8, 61.0)
- added SW2: SW_Push, Button_Switch_THT:SW_PUSH-12mm_Wuerth-430476085716, F.Cu at (139.8, 76.0)
- added SW3: SW_Push, Button_Switch_THT:SW_PUSH_6mm_H5mm, F.Cu at (115.0, 54.0)
- added SW4: SW_SPST, Button_Switch_THT:SW_E-Switch_EG1271_SPDT, F.Cu at (113.5, 109.5)
- added TP1: TestPoint_Probe, TestPoint:TestPoint_Pad_D2.0mm, F.Cu at (117.0, 73.5)
- added TP2: TestPoint_Probe, TestPoint:TestPoint_Pad_D2.0mm, F.Cu at (115.5, 64.5)
- added TP3: TestPoint_Probe, TestPoint:TestPoint_Pad_D2.0mm, F.Cu at (108.5, 64.0)
- added TP4: TestPoint_Probe, TestPoint:TestPoint_Pad_D2.0mm, F.Cu at (105.5, 75.0)
- added TP5: TestPoint_Probe, TestPoint:TestPoint_Pad_D2.0mm, F.Cu at (90.0, 99.0)
- added U1: MAX2650EUS+T, MAX2650EUS+T:21-0052F_MXM, F.Cu at (113.5, 68.4)
- added U2: MAX2650EUS+T, MAX2650EUS+T:21-0052F_MXM, F.Cu at (109.0, 68.4)
- added U5: MIC5219-5.0YM5, Package_TO_SOT_SMD:SOT-23-5, F.Cu at (95.0, 103.4)
- C5: value C -> 470pF
- C6: renamed from C4; value C -> 1uF
- J2: renamed from J1; moved to B.Cu
- R2: renamed from R1; value R -> 10k
- R3: renamed from R2; value R -> 10k
- R4: renamed from R3; value R -> 10k
- moved U6 105.0 mm to (88.0, 84.2), turned to -90 degrees
- moved R4 94.2 mm to (110.5, 55.0), turned to -90 degrees
- moved J1 87.7 mm to (116.8, 94.5), turned to 180 degrees
- moved BT1 74.4 mm to (103.2, 109.5), turned to -90 degrees
- moved C6 69.4 mm to (95.0, 107.0), turned to 180 degrees
- moved AFF2 67.9 mm to (130.3, 47.5)
- moved R10 67.9 mm to (138.0, 43.5)
- moved R13 67.9 mm to (118.5, 43.5)
- moved R14 67.9 mm to (133.0, 43.5)
- moved R15 67.9 mm to (116.0, 43.5)
- moved R16 67.9 mm to (130.5, 43.5)
- moved R17 67.9 mm to (118.5, 36.0)
- moved R18 67.9 mm to (133.0, 36.0)
- moved R19 67.9 mm to (116.0, 36.0)
- moved R20 67.9 mm to (130.5, 36.0)
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- renumbered C1 to C3, C2 to C4, J2 to J1, R9 to R10, R10 to R13, R11 to R14, R12 to R15, R13 to R16, R14 to R17, R15 to R18, R16 to R19, R17 to R20, R18 to R21, R19 to R22, R4 to R5, R5 to R6, R6 to R7, R7 to R8, R8 to R9, U1 to U3, U2 to U4, U3 to U6
Connections:
- BT1 pad 1: ENTROPY -> +9V
- C5 pad 1: +5V -> Net-(U2-OUT)
- C5 pad 2: GND -> ENTROPY
Routing:
- net GND: track 0.00 -> 225.8 mm, vias 0 -> 3
- net +5V: track 5.04 -> 81.4 mm, vias 0 -> 2
- net Net-(U4-QH): track 0.00 -> 60.0 mm
- net OUT_CLK1: track 0.00 -> 59.1 mm
- net SHIFT_IN1: track 0.00 -> 56.5 mm
- net CLK1: track 0.00 -> 56.3 mm, vias 0 -> 1
- net CLR1: track 0.00 -> 56.1 mm
- net Net-(U3-QH): track 0.71 -> 54.2 mm
- net RESET: track 0.00 -> 50.7 mm
- net Net-(U4-QA): track 0.00 -> 46.1 mm, vias 0 -> 1
- net Net-(U4-QG): track 0.00 -> 44.8 mm, vias 0 -> 1
- net Net-(U4-QF): track 0.00 -> 44.7 mm, vias 0 -> 1
- net Net-(U4-QB): track 0.00 -> 44.2 mm, vias 0 -> 2
- net Net-(U4-QC): track 0.00 -> 42.4 mm
- net Net-(U4-QE): track 0.00 -> 37.4 mm, vias 0 -> 1
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Other:
- board outline added: 69.5 x 90.5 mm

Commit message: Finished tracing
Parts:
- removed TP3: TestPoint_Probe, TestPoint:TestPoint_Pad_D2.0mm
- removed the U2 at (109.0, 68.4)
- added EN_RAND: SolderJumper_2_Open, Jumper:SolderJumper-2_P1.3mm_Open_TrianglePad1.0x1.5mm, F.Cu at (102.7, 84.5)
- added REF**: OSHW-Logo_7.5x8mm_SilkScreen, Symbol:OSHW-Logo_7.5x8mm_SilkScreen, F.Cu at (133.0, 109.0)
- CHANGE DICE: renamed from SW1
- LAST RESULT: renamed from SW2
- moved D1 4.50 mm to (105.0, 104.5)
- moved RAW 1.10 mm to (118.0, 73.0)
- renumbered TP5 to 5V, TP4 to ENTROPY, TP2 to INTER, J1 to PROGRAM, R8 to R10, R9 to R11, R10 to R12, R11 to R5, R12 to R6, R5 to R7, R6 to R8, R7 to R9, TP1 to RAW, SW3 to RESET, U3 to U2, U4 to U3, U5 to U4, U6 to U5
Connections:
- BT1 pad 1: +9V -> Net-(BT1-+)
- C5 pad 1: Net-(U2-OUT) -> Net-(U1-OUT)
- C5 pad 2: ENTROPY -> Net-(JP1-A)
- C6 pad 1: Net-(D1-K) -> +9V
- D1 pad 1: Net-(D1-K) -> +9V
- ENTROPY pad 1: ENTROPY -> Net-(JP1-A)
- R5 pad 2: ENTROPY -> Net-(JP1-A)
- R6 pad 1: ENTROPY -> Net-(JP1-A)
- SW4 pad 1: +9V -> Net-(BT1-+)
- SW4 pad 4: +9V -> (no net)
- SW4 pad 5: Net-(D1-A) -> (no net)
- U4 pad 1: Net-(D1-K) -> +9V
- U4 pad 3: Net-(D1-K) -> +9V
Routing:
- net +5V: track 81.4 -> 268.2 mm, vias 2 -> 6
- net GND: track 225.8 -> 383.4 mm, vias 3 -> 4
- net BTN_LAST: track 12.5 -> 60.8 mm, vias 0 -> 2
- net BTN_CH: track 17.7 -> 63.8 mm, vias 0 -> 2
- net SPI_CLK: track 0.00 -> 41.5 mm, vias 0 -> 2
- net SHAKE_OUT: track 0.00 -> 37.9 mm, vias 0 -> 1
- net RESET: track 50.7 -> 86.9 mm, vias 0 -> 1
- net +9V: track 10.5 -> 43.6 mm
- net Net-(JP1-A): track 0.00 -> 20.4 mm
- net Net-(BT1-+): track 0.00 -> 10.5 mm
- net Net-(D1-K): track 9.33 -> 0.00 mm
- net Net-(D1-A): track 12.8 -> 8.29 mm
- net Net-(U2-OUT): track 3.29 -> 0.00 mm
- net Net-(U1-OUT): track 9.54 -> 12.2 mm
- net ENTROPY: track 11.5 -> 9.81 mm
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Other:
- board size 69.5 x 90.5 mm -> 78.5 x 98.5 mm
- board text added: "SHAKE!"
- board text added: "by Jan Wielpütz https://github.com/janWie96/SchuettelDice.git"
