File: Digitaler_Wuerfel.kicad_pcb (KiCad board)
At the start: 2 copper layers, 78.5 x 98.5 mm, 53 parts, among them J2 Conn_01x03_Pin, Q1 2N3904, SW4 SW_SPST, U1 MAX2650EUS+T, U2 74HC595, U3 74HC595, U4 MIC5219-5.0YM5, U5 ATmega328PB-A

Commit message: Added decoupling capacitors and ground plane
Parts:
- added C10: 100nF, Capacitor_SMD:C_0805_2012Metric_Pad1.18x1.45mm_HandSolder, F.Cu at (89.0, 77.0)
- added C9: 100nF, Capacitor_SMD:C_0805_2012Metric_Pad1.18x1.45mm_HandSolder, F.Cu at (89.0, 91.5)
- added REF**: MountingHole_3.2mm_M3_ISO14580, MountingHole:MountingHole_3.2mm_M3_ISO14580, F.Cu at (143.5, 26.5)
- added REF**: MountingHole_3.2mm_M3_ISO14580, MountingHole:MountingHole_3.2mm_M3_ISO14580, F.Cu at (75.3, 114.0)
- added REF**: MountingHole_3.2mm_M3_Pad_Via, MountingHole:MountingHole_3.2mm_M3_Pad_Via, F.Cu at (143.5, 114.0)
- SW1: renamed from CHANGE DICE
- SW2: renamed from LAST RESULT
- moved REF** 4.92 mm to (131.0, 113.5)
- renumbered PROGRAM to J1, RESET to SW3, RAW to TP1, INTER to TP2, ENTROPY to TP3, 5V to TP4, GND to TP5
Connections:
- U5 pad 18: unconnected-(U5-AVCC-Pad18) -> +5V
- U5 pad 20: unconnected-(U5-AREF-Pad20) -> Net-(U5-AREF)
Routing:
- net GND: track 383.4 -> 2.80 mm, vias 4 -> 31
- net +5V: track 268.2 -> 283.5 mm, vias 6 -> 8
- net +9V: track 43.6 -> 56.9 mm, vias 0 -> 2
- net Net-(U5-AREF): track 0.00 -> 3.13 mm
- added copper zone on B.Cu, net GND
- added copper zone on F.Cu, net GND
Other:
- board text added: "5V"
- board text added: "CHANGE DICE"
- board text added: "ENTROPY"
- board text added: "EN_RAND"
- board text added: "GND"
- board text added: "INTER"
- board text added: "LAST RESULT"
- board text added: "RAW"
